File: hardware/securelemakin-board/securelemakin-board.kicad_pcb (KiCad board)
At the start: 2 copper layers, 50 x 76 mm, 6 parts, among them U1 WeMos_S2_mini, U2 Sparkfun_Pro_Micro

Commit message: move unused files
Routing:
- net Earth: track 166.1 -> 166.8 mm
Changed lines of the file:
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@@
   (segment (start 204.870151 106.24) (end 203.2 104.569849) (width 1) (layer "B.Cu") (net 4))
   (segment (start 181.05 111.47) (end 190.21 111.47) (width 1) (layer "B.Cu") (net 5))
-  (segment (start 198.12 50.8) (end 190.5 50.8) (width 1) (layer "B.Cu") (net 5))
+  (segment (start 201.25 50.8) (end 201.45 51) (width 1) (layer "B.Cu") (net 5))
+  (segment (start 190.5 50.8) (end 201.25 50.8) (width 1) (layer "B.Cu") (net 5))
   (segment (start 211.94 111.76) (end 208.28 111.76) (width 1) (layer "B.Cu") (net 5))
   (segment (start 174.55 111.47) (end 181.05 111.47) (width 1) (layer "B.Cu") (net 5))
-  (segment (start 201.45 107.47) (end 205.74 111.76) (width 1) (layer "B.Cu") (net 5))
   (segment (start 193.04 115.9) (end 193.98 116.84) (width 1) (layer "B.Cu") (net 5))
   (segment (start 208.28 111.76) (end 205.74 111.76) (width 1) (layer "B.Cu") (net 5))
-  (segment (start 201.45 54.13) (end 201.45 107.47) (width 1) (layer "B.Cu") (net 5))
-  (segment (start 207.79 47.34137) (end 207.79 44.870862) (width 1) (layer "B.Cu") (net 5))
-  (segment (start 204.673756 43.18) (end 200.66 47.193756) (width 1) (layer "B.Cu") (net 5))
   (segment (start 211.249849 104.14) (end 211.94 104.14) (width 1) (layer "B.Cu") (net 5))
   (segment (start 193.98 116.84) (end 201.219138 116.84) (width 1) (layer "B.Cu") (net 5))
   (segment (start 190.21 111.47) (end 193.04 114.3) (width 1) (layer "B.Cu") (net 5))
-  (segment (start 200.66 48.26) (end 198.12 50.8) (width 1) (layer "B.Cu") (net 5))
   (segment (start 205.74 101.6) (end 208.28 101.6) (width 1) (layer "B.Cu") (net 5))
   (segment (start 208.28 111.76) (end 208.28 107.816955) (width 1) (layer "B.Cu") (net 5))
@@
   (segment (start 218.44 111.76) (end 211.94 111.76) (width 1) (layer "B.Cu") (net 5))
   (segment (start 218.44 104.14) (end 211.94 104.14) (width 1) (layer "B.Cu") (net 5))
-  (segment (start 207.79 44.870862) (end 206.099138 43.18) (width 1) (layer "B.Cu") (net 5))
+  (segment (start 205.74 111.76) (end 201.45 107.47) (width 1) (layer "B.Cu") (net 5))
+  (segment (start 204.673756 43.18) (end 206.099138 43.18) (width 1) (layer "B.Cu") (net 5))
   (segment (start 193.04 114.3) (end 193.04 115.9) (width 1) (layer "B.Cu") (net 5))
-  (segment (start 198.12 50.8) (end 201.45 54.13) (width 1) (layer "B.Cu") (net 5))
   (segment (start 190.5 53.34) (end 190.5 50.8) (width 1) (layer "B.Cu") (net 5))
-  (segment (start 206.099138 43.18) (end 204.673756 43.18) (width 1) (layer "B.Cu") (net 5))
   (segment (start 201.219138 116.84) (end 205.74 112.319138) (width 1) (layer "B.Cu") (net 5))
+  (segment (start 201.45 107.47) (end 201.45 51) (width 1) (layer "B.Cu") (net 5))
   (segment (start 209.4 101.6) (end 208.28 101.6) (width 1) (layer "B.Cu") (net 5))
+  (segment (start 201.45 51) (end 201.45 46.403756) (width 1) (layer "B.Cu") (net 5))
   (segment (start 211.94 104.14) (end 209.4 101.6) (width 1) (layer "B.Cu") (net 5))
-  (segment (start 206.87137 48.26) (end 207.79 47.34137) (width 1) (layer "B.Cu") (net 5))
+  (segment (start 201.45 46.403756) (end 204.673756 43.18) (width 1) (layer "B.Cu") (net 5))
   (segment (start 210.03 106.066955) (end 210.03 105.359849) (width 1) (layer "B.Cu") (net 5))
-  (segment (start 200.66 47.193756) (end 200.66 48.26) (width 1) (layer "B.Cu") (net 5))
+  (segment (start 206.099138 43.18) (end 207.79 44.870862) (width 1) (layer "B.Cu") (net 5))
   (segment (start 210.03 105.359849) (end 211.249849 104.14) (width 1) (layer "B.Cu") (net 5))
-  (segment (start 205.74 48.26) (end 206.87137 48.26) (width 1) (layer "B.Cu") (net 5))
+  (segment (start 206.87137 48.26) (end 205.74 48.26) (width 1) (layer "B.Cu") (net 5))
   (segment (start 205.74 112.319138) (end 205.74 111.76) (width 1) (layer "B.Cu") (net 5))
+  (segment (start 207.79 44.870862) (end 207.79 47.34137) (width 1) (layer "B.Cu") (net 5))
+  (segment (start 207.79 47.34137) (end 206.87137 48.26) (width 1) (layer "B.Cu") (net 5))
   (segment (start 195.58 59.82863) (end 191.63137 55.88) (width 1) (layer "B.Cu") (net 10))
   (segment (start 187.96 91.44) (end 189.162081 91.44) (width 1) (layer "B.Cu") (net 10))
